File: ezLCD-303-PicoPi-Breakout-Board.kicad_pcb (KiCad board)
At the start: 2 copper layers, 71.1 x 50.8 mm, 20 parts, among them J1 ELP-000097, J2 ELP-000029, J3 ELP-000063, J4 ELP-000094, J5 ELP-000094, J6 ELP-000098, J7 ELP-000098, U1 ELP-000052

Commit message: Adjusted origins on the PCB
Other:
- board text added: "0"
- board text added: "0 mm"
- board text added: "0.01 mm"
- board text added: "0.02"
- board text added: "0.035 mm"
- board text added: "1"
- board text added: "1.51 mm"
- board text added: "3.3"
- board text added: "4.5"
- board text added: "B.Cu"
- board text added: "B.Mask"
- board text added: "B.Paste"
- board text added: "B.Silkscreen"
- board text added: "Bottom Silk Screen"
- board text added: "Bottom Solder Mask"
- board text added: "Bottom Solder Paste"
- board text added: "Color"
- board text added: "Dielectric"
- board text added: "Epsilon R"
- board text added: "F.Cu"
- board text added: "F.Mask"
- board text added: "F.Paste"
- board text added: "F.Silkscreen"
- board text added: "FR4"
- board text added: "Layer Name"
- board text added: "Loss Tangent"
- board text added: "Material"
- board text added: "Not specified"
- board text added: "Thickness (mm)"
- board text added: "Top Silk Screen"
- board text added: "Top Solder Mask"
- board text added: "Top Solder Paste"
- board text added: "Type"
- board text added: "copper"
- board text added: "core"

Commit message: Added additional silk to help indicate connection points.
Other:
- board text added: "0.0000 mm / 0.0000 mm"
- board text added: "0.3000 mm"
- board text added: "1-B/Z 2-A/Y"
- board text added: "1-VBUS 2-GND"
- board text added: "1-VSYS 2-GND"
- board text added: "1.6000 mm"
- board text added: "10"
- board text added: "2"
- board text added: "71.1200 mm x 50.8000 mm"
- board text added: "BOARD CHARACTERISTICS"
- board text added: "Board Thickness:"
- board text added: "Board overall dimensions:"
- board text added: "Castellated pads:"
- board text added: "Copper Finish:"
- board text added: "Copper Layer Count:"
- board text added: "Edge card connectors:"
- board text added: "Impedance Control:"
- board text added: "Min hole diameter:"
- board text added: "Min track/spacing:"
- board text added: "No"
- board text added: "None"
- board text added: "Plated Board Edge:"
Changed lines of the file:
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@@
   (gr_rect (start 90.52 49.5) (end 161.64 100.3)
     (stroke (width 0.1) (type default)) (fill none) (layer "Edge.Cuts"))
+  (gr_text "1-B/Z\n2-A/Y" (at 148.559 92.045) (layer "F.SilkS")
+    (effects (font (size 1 1) (thickness 0.15)) (justify left bottom))
+  )
+  (gr_text "1" (at 97.505 59.279) (layer "F.SilkS")
+    (effects (font (size 1 1) (thickness 0.15)) (justify left bottom))
+  )
+  (gr_text "1-VSYS\n2-GND" (at 91.536 91.537) (layer "F.SilkS")
+    (effects (font (size 1 1) (thickness 0.15)) (justify left bottom))
+  )
   (gr_text "QUAD\nENCD" (at 155.067 87.63) (layer "F.SilkS")
     (effects (font (size 1.5 1.5) (thickness 0.3) bold) (justify left bottom))
   )
+  (gr_text "1-VBUS\n2-GND" (at 91.028 61.057) (layer "F.SilkS")
+    (effects (font (size 1 1) (thickness 0.15)) (justify left bottom))
+  )
+  (gr_text "1" (at 146.146 95.982) (layer "F.SilkS")
+    (effects (font (size 1 1) (thickness 0.15)) (justify left bottom))
+  )
+  (gr_text "2" (at 97.505 91.029) (layer "F.SilkS")
+    (effects (font (size 1 1) (thickness 0.15)) (justify left bottom))
+  )
+  (gr_text "10" (at 146.019 57.628) (layer "F.SilkS")
+    (effects (font (size 1 1) (thickness 0.15)) (justify left bottom))
+  )
   (gr_text "B.Paste" (at 36.787 168.7) (layer "Dwgs.User")
     (effects (font (size 1.5 1.5) (thickness 0.1)) (justify left top))
@@
     (effects (font (size 1.5 1.5) (thickness 0.1)) (justify left top))
   )
+  (gr_text "No" (at 129.064138 128.661) (layer "Dwgs.User")
+    (effects (font (size 1.5 1.5) (thickness 0.2)) (justify left top))
+  )
+  (gr_text "" (at 129.064138 116.79) (layer "Dwgs.User")
+    (effects (font (size 1.5 1.5) (thickness 0.2)) (justify left top))
+  )
+  (gr_text "0.0000 mm / 0.0000 mm" (at 69.964143 120.747) (layer "Dwgs.User")
+    (effects (font (size 1.5 1.5) (thickness 0.2)) (justify left top))
+  )
   (gr_text "0" (at 143.158431 143.458) (layer "Dwgs.User")
     (effects (font (size 1.5 1.5) (thickness 0.1)) (justify left top))
@@
     (effects (font (size 1.5 1.5) (thickness 0.1)) (justify left top))
   )
+  (gr_text "2" (at 69.964143 112.833) (layer "Dwgs.User")
+    (effects (font (size 1.5 1.5) (thickness 0.2)) (justify left top))
+  )
+  (gr_text "Board overall dimensions: " (at 37.307 116.79) (layer "Dwgs.User")
+    (effects (font (size 1.5 1.5) (thickness 0.2)) (justify left top))
+  )
   (gr_text "0.01 mm" (at 93.744143 165.094) (layer "Dwgs.User")
     (effects (font (size 1.5 1.5) (thickness 0.1)) (justify left top))
@@
     (effects (font (size 1.5 1.5) (thickness 0.1)) (justify left top))
   )
+  (gr_text "Castellated pads: " (at 37.307 128.661) (layer "Dwgs.User")
+    (effects (font (size 1.5 1.5) (thickness 0.2)) (justify left top))
+  )
   (gr_text "1.51 mm" (at 93.744143 157.882) (layer "Dwgs.User")
     (effects (font (size 1.5 1.5) (thickness 0.1)) (justify left top))
   )
+  (gr_text "0.3000 mm" (at 129.064138 120.747) (layer "Dwgs.User")
+    (effects (font (size 1.5 1.5) (thickness 0.2)) (justify left top))
+  )
   (gr_text "1" (at 130.272716 143.458) (layer "Dwgs.User")
     (effects (font (size 1.5 1.5) (thickness 0.1)) (justify left top))
@@
     (effects (font (size 1.5 1.5) (thickness 0.1)) (justify left top))
   )
+  (gr_text "Copper Layer Count: " (at 37.307 112.833) (layer "Dwgs.User")
+    (effects (font (size 1.5 1.5) (thickness 0.2)) (justify left top))
+  )
   (gr_text "Epsilon R" (at 130.272716 139.15) (layer "Dwgs.User")
     (effects (font (size 1.5 1.5) (thickness 0.3)) (justify left top))
@@
     (effects (font (size 1.5 1.5) (thickness 0.1)) (justify left top))
   )
+  (gr_text "71.1200 mm x 50.8000 mm" (at 69.964143 116.79) (layer "Dwgs.User")
+    (effects (font (size 1.5 1.5) (thickness 0.2)) (justify left top))
+  )
+  (gr_text "1.6000 mm" (at 129.064138 112.833) (layer "Dwgs.User")
+    (effects (font (size 1.5 1.5) (thickness 0.2)) (justify left top))
+  )
   (gr_text "B.Cu" (at 36.787 161.488) (layer "Dwgs.User")
     (effects (font (size 1.5 1.5) (thickness 0.1)) (justify left top))
   )
+  (gr_text "No" (at 69.964143 128.661) (layer "Dwgs.User")
+    (effects (font (size 1.5 1.5) (thickness 0.2)) (justify left top))
+  )
   (gr_text "F.Cu" (at 36.787 154.276) (layer "Dwgs.User")
     (effects (font (size 1.5 1.5) (thickness 0.1)) (justify left top))
   )
+  (gr_text "No" (at 69.964143 132.618) (layer "Dwgs.User")
+    (effects (font (size 1.5 1.5) (thickness 0.2)) (justify left top))
+  )
+  (gr_text "" (at 104.121281 116.79) (layer "Dwgs.User")
+    (effects (font (size 1.5 1.5) (thickness 0.2)) (justify left top))
+  )
   (gr_text "0" (at 143.158431 150.67) (layer "Dwgs.User")
     (effects (font (size 1.5 1.5) (thickness 0.1)) (justify left top))
@@
     (effects (font (size 1.5 1.5) (thickness 0.1)) (justify left top))
   )
+  (gr_text "Board Thickness: " (at 104.121281 112.833) (layer "Dwgs.User")
+    (effects (font (size 1.5 1.5) (thickness 0.2)) (justify left top))
+  )
   (gr_text "1" (at 130.272716 172.306) (layer "Dwgs.User")
     (effects (font (size 1.5 1.5) (thickness 0.1)) (justify left top))
@@
     (effects (font (size 1.5 1.5) (thickness 0.1)) (justify left top))
   )
+  (gr_text "Copper Finish: " (at 37.307 124.704) (layer "Dwgs.User")
+    (effects (font (size 1.5 1.5) (thickness 0.2)) (justify left top))
+  )
   (gr_text "0 mm" (at 93.744143 168.7) (layer "Dwgs.User")
     (effects (font (size 1.5 1.5) (thickness 0.1)) (justify left top))
@@
     (effects (font (size 1.5 1.5) (thickness 0.1)) (justify left top))
   )
+  (gr_text "Min track/spacing: " (at 37.307 120.747) (layer "Dwgs.User")
+    (effects (font (size 1.5 1.5) (thickness 0.2)) (justify left top))
+  )
+  (gr_text "Min hole diameter: " (at 104.121281 120.747) (layer "Dwgs.User")
+    (effects (font (size 1.5 1.5) (thickness 0.2)) (justify left top))
+  )
   (gr_text "" (at 113.772715 168.7) (layer "Dwgs.User")
     (effects (font (size 1.5 1.5) (thickness 0.1)) (justify left top))
@@
     (effects (font (size 1.5 1.5) (thickness 0.1)) (justify left top))
   )
+  (gr_text "No" (at 129.064138 124.704) (layer "Dwgs.User")
+    (effects (font (size 1.5 1.5) (thickness 0.2)) (justify left top))
+  )
+  (gr_text "BOARD CHARACTERISTICS" (at 36.557 107.339) (layer "Dwgs.User")
+    (effects (font (size 2 2) (thickness 0.4)) (justify left top))
+  )
   (gr_text "Not specified" (at 77.244142 150.67) (layer "Dwgs.User")
     (effects (font (size 1.5 1.5) (thickness 0.1)) (justify left top))
@@
     (effects (font (size 1.5 1.5) (thickness 0.3)) (justify left top))
   )
+  (gr_text "Impedance Control: " (at 104.121281 124.704) (layer "Dwgs.User")
+    (effects (font (size 1.5 1.5) (thickness 0.2)) (justify left top))
+  )
   (gr_text "Color" (at 113.772715 139.15) (layer "Dwgs.User")
     (effects (font (size 1.5 1.5) (thickness 0.3)) (justify left top))
   )
+  (gr_text "None" (at 69.964143 124.704) (layer "Dwgs.User")
+    (effects (font (size 1.5 1.5) (thickness 0.2)) (justify left top))
+  )
+  (gr_text "Edge card connectors: " (at 37.307 132.618) (layer "Dwgs.User")
+    (effects (font (size 1.5 1.5) (thickness 0.2)) (justify left top))
+  )
   (gr_text "copper" (at 52.172714 161.488) (layer "Dwgs.User")
     (effects (font (size 1.5 1.5) (thickness 0.1)) (justify left top))
@@
   (gr_text "FR4" (at 77.244142 157.882) (layer "Dwgs.User")
     (effects (font (size 1.5 1.5) (thickness 0.1)) (justify left top))
+  )
+  (gr_text "Plated Board Edge: " (at 104.121281 128.661) (layer "Dwgs.User")
+    (effects (font (size 1.5 1.5) (thickness 0.2)) (justify left top))
   )
   (gr_text "Type" (at 52.172714 139.15) (layer "Dwgs.User")
@@
   (segment (start 150.44 50.72) (end 151.257 50.72) (width 0.25) (layer "F.Cu") (net 58))
   (segment (start 151.257 50.72) (end 153.06 52.523) (width 0.508) (layer "F.Cu") (net 58))
+  (group "group-boardCharacteristics" (id 5966067d-beef-4ee7-b1f9-b82bd9f7e3d0)
+    (members
+      0d8d1d79-9477-4ea0-a983-7e3b44aed3ff
+      11aad5b7-9d2e-4325-befc-bb1a885fe999
+      18e8904a-d950-4b49-9734-1e5f67ac875b
+      36bd48b6-3f7e-4f98-805d-ced733707e8c
+      37157a4a-c269-428c-8670-82650d750462
+      4fc68c78-d64a-4a3c-9f5e-3e69a855239d
+      53e409e7-d229-449b-9432-65a6e76f1701
+      6834dd76-713d-4bb8-9d7e-ad685e21073d
+      81f9aa35-4eff-4971-8afe-a9da875fede3
+      840e9fcb-d140-4b20-b287-e31f19204931
+      861a0a3d-b305-4876-b0be-f6e35ea93ebb
+      9d5a4fcb-905e-4167-840a-ce491df4dd93
+      9e24af90-4d5a-4ee6-9484-4d96983d3d26
+      a39cf3b2-0d26-4a1a-b858-3fd062fe69e4
+      aa1d02b5-726d-47b0-92fb-dc0a8be1b6ff
+      ba8b8c7b-faf9-44e2-8915-76c4c813b4fb
+      bb765937-9169-43cb-8fdb-ff6005dc544a
+      c3894182-41c5-497d-8080-e2576700f66a
+      c6a4d1bd-eadd-433e-9f24-95e3930bedcf
+      e1873007-2129-471c-a301-827cfe73245c
+      e72cc176-fe36-4672-9ce3-8767128332ca
+      e87a19de-a011-4090-a0da-9d79cd2a61d0
+      f9e966c5-db9d-4e03-b244-971c420dbc3d
+    )
+  )
   (group "group-boardStackUp" (id e2fb59de-d735-402f-aad2-31247cce35d8)
     (members
