File: top-pico-pi-w.kicad_sch (KiCad schematic)
At the start: 9 parts, among them J4 ELP-000094, J5 ELP-000094, J6 ELP-000098, J7 ELP-000098

Commit message: Fixed errors on the schematic found after fabrication of the X1 PCB's.
Connections:
- net VSYS: no longer J4.1
- net +3.3V: now reaches PCBA1.36 (3V3(OUT))
- net +3.3V: now also J4.1
- no-connect marks 4 -> 3
Changed lines of the file:
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@@
   (junction (at 77.47 116.84) (diameter 0) (color 0 0 0 0)
   )
-  (no_connect (at 186.69 81.28))
   (no_connect (at 186.69 83.82))
   (no_connect (at 186.69 78.74))
@@
     (stroke (width 0) (type default))
   )
+  (wire (pts (xy 203.2 81.28) (xy 186.69 81.28))
+    (stroke (width 0) (type default))
+  )
   (wire (pts (xy 186.69 88.9) (xy 200.66 88.9))
     (stroke (width 0) (type default))
@@
     (stroke (width 0) (type default))
   )
-  (wire (pts (xy 60.96 78.74) (xy 58.42 78.74))
+  (wire (pts (xy 58.42 78.74) (xy 64.77 78.74))
     (stroke (width 0) (type default))
   )
@@
     (stroke (width 0) (type default))
   )
+  (wire (pts (xy 203.2 64.77) (xy 203.2 81.28))
+    (stroke (width 0) (type default))
+  )
   (wire (pts (xy 213.36 83.82) (xy 227.33 83.82))
     (stroke (width 0) (type default))
@@
   )
   (wire (pts (xy 186.69 109.22) (xy 199.39 109.22))
+    (stroke (width 0) (type default))
+  )
+  (wire (pts (xy 64.77 66.04) (xy 64.77 78.74))
     (stroke (width 0) (type default))
   )
@@
     (property "Intersheetrefs" "${INTERSHEET_REFS}" (at 64.4042 96.52 0)
       (effects (font (size 1.27 1.27)) (justify right) hide)
-    )
-  )
-  (global_label "VSYS" (shape input) (at 60.96 78.74 0) (fields_autoplaced)
-    (effects (font (size 1.27 1.27)) (justify left))
-    (property "Intersheetrefs" "${INTERSHEET_REFS}" (at 68.462 78.74 0)
-      (effects (font (size 1.27 1.27)) (justify left) hide)
     )
   )
@@
         )
       )
+    )
+  )
+  (symbol (lib_id "power:+3.3V") (at 64.77 66.04 0) (unit 1)
+    (in_bom yes) (on_board yes) (dnp no) (fields_autoplaced)
+    (property "Reference" "#PWR04" (at 64.77 69.85 0)
+      (effects (font (size 1.27 1.27)) hide)
+    )
+    (property "Value" "+3.3V" (at 64.77 60.96 0)
+      (effects (font (size 1.27 1.27)))
+    )
+    (property "Footprint" "" (at 64.77 66.04 0)
+      (effects (font (size 1.27 1.27)) hide)
+    )
+    (property "Datasheet" "" (at 64.77 66.04 0)
+      (effects (font (size 1.27 1.27)) hide)
+    )
+    (pin "1")
+    (instances
+      (project "ezLCD-303-PicoPi-Breakout-Board"
+        (path "/00955ca7-e382-491b-9e67-f8c537447774/107ae0b7-6f32-49a5-aebd-43a6142a295e"
+          (reference "#PWR04") (unit 1)
+        )
+        (path "/00955ca7-e382-491b-9e67-f8c537447774/b88a05e9-0a80-4ae1-834b-75c31c8ce3bc"
+          (reference "#PWR014") (unit 1)
+        )
+      )
+      (project "PCB-2301"
+        (path "/1ded335d-6d13-4ffa-94d5-e15dc2cb695c/d4a07de9-06a8-4cb3-8ea5-718fa4e90a32"
+          (reference "#PWR0234") (unit 1)
+        )
+      )
+    )
+  )
+  (symbol (lib_id "power:+3.3V") (at 203.2 64.77 0) (unit 1)
+    (in_bom yes) (on_board yes) (dnp no) (fields_autoplaced)
+    (property "Reference" "#PWR04" (at 203.2 68.58 0)
+      (effects (font (size 1.27 1.27)) hide)
+    )
+    (property "Value" "+3.3V" (at 203.2 59.69 0)
+      (effects (font (size 1.27 1.27)))
+    )
+    (property "Footprint" "" (at 203.2 64.77 0)
+      (effects (font (size 1.27 1.27)) hide)
+    )
+    (property "Datasheet" "" (at 203.2 64.77 0)
+      (effects (font (size 1.27 1.27)) hide)
+    )
+    (pin "1")
+    (instances
+      (project "ezLCD-303-PicoPi-Breakout-Board"
+        (path "/00955ca7-e382-491b-9e67-f8c537447774/107ae0b7-6f32-49a5-aebd-43a6142a295e"
+          (reference "#PWR04") (unit 1)
+        )
+        (path "/00955ca7-e382-491b-9e67-f8c537447774/b88a05e9-0a80-4ae1-834b-75c31c8ce3bc"
+          (reference "#PWR05") (unit 1)
+        )
+      )
+      (project "PCB-2301"
+        (path "/1ded335d-6d13-4ffa-94d5-e15dc2cb695c/d4a07de9-06a8-4cb3-8ea5-718fa4e90a32"
+          (reference "#PWR0234") (unit 1)
+        )
+      )
